Commit message: Updated robot.xacro to include wheels

File: urdf/robot.xacro (robot description, xacro)
@@ -75,9 +75,23 @@
         </collision>
     </link>
+    <link name = "wheel_center">
+        <visual>
+            <origin xyz = "0.0 0.0 0.0" rpy = "${-1*pi/2} 0.0 0.0" />
+            <geometry>
+                <cylinder radius="0.15" length="0.05" />
+            </geometry>
+        </visual>
+        <collision>
+            <origin xyz = "0.0 0.0 0.0" rpy = "${-1*pi/2} 0.0 0.0" />
+            <geometry>
+                <cylinder radius="0.15" length="0.05" />
+            </geometry>
+        </collision>
+    </link>
     <!-- XACRO Macro definition block to add around the wheel link and joint !-->
     <xacro:macro name = "xacro_name" params = "side reflect" >
-        <link name = "wheel_left">
+        <link name = "wheel_${side}">
             <visual>
-                <origin xyz = "-0.10 0.4 0.0" rpy = "-1.5707 0.0 0.0" />
+                <origin xyz = "-0.10 0 0.0" rpy = "${-1*pi/2} 0.0 0.0" />
                 <geometry>
                     <cylinder radius="0.2" length="0.05" />
@@ -85,5 +99,5 @@
             </visual>
             <collision>
-                <origin xyz = "-0.10 0.4 0.0" rpy = "-1.5707 0.0 0.0" />
+                <origin xyz = "-0.10 0 0.0" rpy = "${-1*pi/2} 0.0 0.0" />
                 <geometry>
                     <cylinder radius="0.2" length="0.05" />
@@ -91,12 +105,18 @@
             </collision>
         </link>
-        <joint name = "base_wheel_left_joint" type = "fixed" >
+        <joint name = "base_wheel_${side}_joint" type = "fixed" >
             <parent link = "base" />
-            <child link = "wheel_left" />
-            <origin xyz = "0 0 0" rpy = "0 0 0" />
+            <child link = "wheel_${side}" />
+            <origin xyz = "0 ${reflect * 0.4} 0" />
         </joint >
     </xacro:macro >
     <!-- Call the XACRO Macro. It should be the left wheel !-->
     <xacro:xacro_name side = "left" reflect = "1" />
+    <xacro:xacro_name side = "right" reflect = "-1" />
+    <joint name = "base_wheel_center_joint" type = "fixed" >
+        <parent link = "base" />
+        <child link = "wheel_center" />
+        <origin xyz = "0.225 0 -0.05" rpy = "0 0 0" />
+    </joint >
     <joint name = "base_laser_vert_bottom_joint" type = "fixed" >
         <parent link = "base" />

Commit message: Updated robot.xacro for contious joints for wheels

File: urdf/robot.xacro (robot description, xacro)
@@ -93,5 +93,5 @@
         <link name = "wheel_${side}">
             <visual>
-                <origin xyz = "-0.10 0 0.0" rpy = "${-1*pi/2} 0.0 0.0" />
+                <origin xyz = "0 0 0.0" rpy = "${-1*pi/2} 0.0 0.0" />
                 <geometry>
                     <cylinder radius="0.2" length="0.05" />
@@ -99,5 +99,5 @@
             </visual>
             <collision>
-                <origin xyz = "-0.10 0 0.0" rpy = "${-1*pi/2} 0.0 0.0" />
+                <origin xyz = "0 0 0.0" rpy = "${-1*pi/2} 0.0 0.0" />
                 <geometry>
                     <cylinder radius="0.2" length="0.05" />
@@ -105,8 +105,9 @@
             </collision>
         </link>
-        <joint name = "base_wheel_${side}_joint" type = "fixed" >
+        <joint name = "base_wheel_${side}_joint" type = "continuous" >
             <parent link = "base" />
             <child link = "wheel_${side}" />
-            <origin xyz = "0 ${reflect * 0.4} 0" />
+            <origin xyz = "-0.10 ${reflect * 0.4} 0" />
+            <axis xyz = " 0.0 1.0 0.0" />
         </joint >
     </xacro:macro >
@@ -114,8 +115,9 @@
     <xacro:xacro_name side = "left" reflect = "1" />
     <xacro:xacro_name side = "right" reflect = "-1" />
-    <joint name = "base_wheel_center_joint" type = "fixed" >
+    <joint name = "base_wheel_center_joint" type = "continuous" >
         <parent link = "base" />
         <child link = "wheel_center" />
         <origin xyz = "0.225 0 -0.05" rpy = "0 0 0" />
+        <axis xyz = " 0.0 1.0 0.0" />
     </joint >
     <joint name = "base_laser_vert_bottom_joint" type = "fixed" >

Commit message: Updated robot.xacro with sensor meshes

File: urdf/robot.xacro (robot description, xacro)
@@ -18,61 +18,27 @@
         </collision>
     </link>
-    <!-- Changed name from laser_vert_bottom_joint as it is not a joint !-->
-    <link name = "laser_vert_bottom">
-        <visual>
-            <origin xyz = "0.3158 -0.0021 0.5100" rpy = "3.1355 -1.3045 0.0025" />
-            <geometry>
-                <box size = "0.062 0.062 0.087" />
-            </geometry>
-        </visual>
-        <collision>
-            <origin xyz = "0.3158 -0.0021 0.5100" rpy = "3.1355 -1.3045 0.0025" />
-            <geometry>
-                <box size = "0.062 0.062 0.087" />
-            </geometry>
-        </collision>
-    </link>
-    <link name = "laser_vert_top_right">
-        <visual>
-            <origin xyz = "0.2978 -0.1450 1.8451" rpy = "-1.1760 0.6313 -1.9377" />
-            <geometry>
-                <box size = "0.062 0.062 0.087" />
-            </geometry>
-        </visual>
-        <collision>
-            <origin xyz = "0.2978 -0.1450 1.8451" rpy = "-1.1760 0.6313 -1.9377" />
-            <geometry>
-                <box size = "0.062 0.062 0.087" />
-            </geometry>
-        </collision>
-    </link>
-    <link name = "laser_vert_top_left">
-        <visual>
-            <origin xyz = "0.2997 0.1531 1.8443" rpy = "1.1780 0.6198 1.9560" />
-            <geometry>
-                <box size = "0.062 0.062 0.087" />
-            </geometry>
-        </visual>
-        <collision>
-            <origin xyz = "0.2997 0.1531 1.8443" rpy = "1.1780 0.6198 1.9560" />
-            <geometry>
-                <box size = "0.062 0.062 0.087" />
-            </geometry>
-        </collision>
-    </link>
-    <link name = "laser_horiz">
-        <visual>
-            <origin xyz = "0.2325 0.0001 1.9201" rpy = "-0.0012 0.1146 -0.0015" />
-            <geometry>
-                <cylinder radius="0.052" length="0.072" />
-            </geometry>
-        </visual>
-        <collision>
-            <origin xyz = "0.2325 0.0001 1.9201" rpy = "-0.0012 0.1146 -0.0015" />
-            <geometry>
-                <cylinder radius="0.052" length="0.072" />
-            </geometry>
-        </collision>
-    </link>
+     <!-- Include the XACRO file that defines a Hokuyo LIDAR. -->
+    <xacro:include filename = "$(find gazebo_plugins)/test/multi_robot_scenario/xacro/laser/hokuyo.xacro" />
+    <xacro:laser name = "laser_vert_bottom" parent = "base" xyz = "0.3157894464801903 -0.002068548615034871 0.5099999434059285" rpy = "3.1354753 -1.3045001 0.0024658"
+        meshes = "package://gazebo_plugins/test/multi_robot_scenario/meshes/laser" />
+    <!-- XACRO Macro definition block to add around the laser_vert_top !-->
+    <xacro:macro name = "laser_vert_top" params = "side reflect" >
+        <xacro:include filename = "$(find gazebo_plugins)/test/multi_robot_scenario/xacro/laser/hokuyo.xacro" />
+        <xacro:laser name = "laser_vert_top_${side}" parent = "base"
+        xyz = "0.2978 ${reflect *0.1450} 1.8451"
+        rpy = "${reflect *1.1760} 0.6313 ${reflect *1.9377}"
+        meshes = "package://gazebo_plugins/test/multi_robot_scenario/meshes/laser" />
+    </xacro:macro >
+    <!-- Call the XACRO Macro. !-->
+    <xacro:laser_vert_top side = "left" reflect = "1" />
+    <xacro:laser_vert_top side = "right" reflect = "-1" />
+    <!-- Include the XACRO file that defines a Hokuyo LIDAR. -->
+    <xacro:include filename = "$(find velodyne_description)/urdf/VLP-16.urdf.xacro" />
+    <!-- Invoke the macro to define the Hokuyo LIDAR. -->
+    <xacro:VLP-16 parent = "base" name = "laser_horiz" topic = "laser_horiz/packets" hz = "10"
+        samples = "440" gpu = "false" >
+    <origin xyz = "0.2325416305773505 -0.0001380069427607134 1.920122926231907"
+        rpy = "-0.0012068 0.114646 -0.0015308" />
+    </xacro:VLP-16 >
     <link name = "wheel_center">
         <visual>
@@ -90,5 +56,5 @@
     </link>
     <!-- XACRO Macro definition block to add around the wheel link and joint !-->
-    <xacro:macro name = "xacro_name" params = "side reflect" >
+    <xacro:macro name = "wheels" params = "side reflect" >
         <link name = "wheel_${side}">
             <visual>
@@ -112,7 +78,7 @@
         </joint >
     </xacro:macro >
-    <!-- Call the XACRO Macro. It should be the left wheel !-->
-    <xacro:xacro_name side = "left" reflect = "1" />
-    <xacro:xacro_name side = "right" reflect = "-1" />
+    <!-- Call the XACRO Macro. !-->
+    <xacro:wheels side = "left" reflect = "1" />
+    <xacro:wheels side = "right" reflect = "-1" />
     <joint name = "base_wheel_center_joint" type = "continuous" >
         <parent link = "base" />
@@ -121,24 +87,3 @@
         <axis xyz = " 0.0 1.0 0.0" />
     </joint >
-    <joint name = "base_laser_vert_bottom_joint" type = "fixed" >
-        <parent link = "base" />
-        <!-- Changed name from laser_vert_bottom_joint as it is not a joint !-->
-        <child link = "laser_vert_bottom" />
-        <origin xyz = "0 0 0" rpy = "0 0 0" />
-    </joint >
-    <joint name = "base_laser_vert_top_right_joint" type = "fixed" >
-        <parent link = "base" />
-        <child link = "laser_vert_top_right" />
-        <origin xyz = "0 0 0" rpy = "0 0 0" />
-    </joint >
-    <joint name = "base_laser_vert_top_left_joint" type = "fixed" >
-        <parent link = "base" />
-        <child link = "laser_vert_top_left" />
-        <origin xyz = "0 0 0" rpy = "0 0 0" />
-    </joint >
-        <joint name = "base_laser_horiz_joint" type = "fixed" >
-        <parent link = "base" />
-        <child link = "laser_horiz" />
-        <origin xyz = "0 0 0" rpy = "0 0 0" />
-    </joint >
 </robot>
